File: kicad/keyboard.kicad_pcb (KiCad board)
At the start: 2 copper layers, 288.1 x 97.6 mm, 161 parts, among them J2 USB_C_Receptacle_USB2.0_16P, SW1 SW_Push, SW10 SW_Push, SW11 SW_Push, SW12 SW_Push, SW13 SW_Push, SW14 SW_Push, SW15 SW_Push, SW16 SW_Push, SW17 SW_Push, SW18 SW_Push, SW19 SW_Push, SW2 SW_Push, SW20 SW_Push, SW21 SW_Push, SW22 SW_Push, SW23 SW_Push, SW24 SW_Push, SW25 SW_Push, SW26 SW_Push, SW27 SW_Push, SW28 SW_Push, SW29 SW_Push, SW3 SW_Push, SW30 SW_Push, SW31 SW_Push, SW32 SW_Push, SW33 SW_Push, SW34 SW_Push, SW35 SW_Push, SW36 SW_Push, SW37 SW_Push, SW38 SW_Push, SW39 SW_Push, SW4 SW_Push, SW40 SW_Push, SW41 SW_Push, SW42 SW_Push, SW43 SW_Push, SW44 SW_Push, SW45 SW_Push, SW46 SW_Push, SW47 SW_Push, SW48 SW_Push, SW49 SW_Push, SW5 SW_Push, SW50 SW_Push, SW51 SW_Push, SW52 SW_Push, SW53 SW_Push, SW54 SW_Push, SW55 SW_Push, SW56 SW_Push, SW57 SW_Push, SW58 SW_Push, SW59 SW_Push, SW6 SW_Push, SW60 SW_Push, SW61 SW_Push, SW62 SW_SPST, SW7 SW_Push, SW8 SW_Push, SW9 SW_Push, U4 NCP1117-3.3_SOT223, U5 W25Q128JVS, U6 RP2040, Y2 ABM8-272-T3

Commit message: chore: resize pcb paper
Parts:
- moved D40 71.9 mm to (294.1, 146.4)
- moved C27 71.9 mm to (219.7, 184.1)
- moved D34 71.9 mm to (179.8, 146.4)
- moved D36 71.9 mm to (217.9, 146.4)
- moved D39 71.9 mm to (275.0, 146.4)
- moved D57 71.9 mm to (191.7, 184.5)
- moved D58 71.9 mm to (263.1, 184.5)
- moved D59 71.9 mm to (286.9, 184.5)
- moved REF** 71.9 mm to (329.8, 101.2)
- moved SW14 71.9 mm to (329.8, 101.2)
- moved SW47 71.9 mm to (191.7, 158.4)
- moved SW49 71.9 mm to (229.8, 158.4)
- moved SW52 71.9 mm to (286.9, 158.4)
- moved U5 71.9 mm to (176.4, 177.4)
- moved U6 71.9 mm to (224.3, 177.9)
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